File: kicad/drako-cyberstorm/drako-cyberstorm.kicad_pcb (KiCad board)
At the start: 2 copper layers, 75 x 57 mm, 6 parts, among them U1 Raspberry Pi Pico2, U2 AT28C64B-15PU, U3 SN74HC595N (HIGH-BYTE), U4 SN74HC595N (LOW-BYTE)

Commit message: Finalized Schematic and PCB
Moved shift registers' OE to GPIO 27 and edited the footprint silkscreen to better fit Louisiana Tech's CyberStorm event.
Parts:
- Dual-7-Seg1: value Dual 7-Segment Display -> ~
- R1: value 250 -> 250Ω
- U1: value Raspberry Pi Pico2 -> Pico
Connections:
- U1 pad 32: unconnected-(U1-GPIO27_ADC1-Pad32) -> Net-(U1-GPIO27_ADC1)
- U3 pad 13: /DATA0 -> Net-(U1-GPIO27_ADC1)
- U4 pad 13: /DATA0 -> Net-(U1-GPIO27_ADC1)
Routing:
- net /DATA0: track 131.9 -> 52.1 mm
- net Net-(U1-GPIO27_ADC1): track 0.00 -> 73.1 mm, vias 0 -> 1
Other:
- board text added: "CYBERSTORM: DRAKO"
- board text removed: "The_Goldfish"
