File: kicad/drako-cyberstorm/drako-cyberstorm.kicad_sch (KiCad schematic)
At the start: 6 parts, among them U1 Pico, U2 AT28C64B-15PU, U3 SN74HC595N (HIGH-BYTE), U4 SN74HC595N (LOW-BYTE)

Commit message: Finalized Schematic and PCB
Moved shift registers' OE to GPIO 27 and edited the footprint silkscreen to better fit Louisiana Tech's CyberStorm event.
Parts:
- R1: value 250Ω -> 47Ω
Connections:
- net Address Bus: now also U1.32 (GPIO27_ADC1), U3.13 (~{OE}), U4.13 (~{OE})
- net DATA0: no longer U3.13 (~{OE}), U4.13 (~{OE})
Other:
- company: Quarter Project -> (none)
- title: Drako -> Drako Hardware Challenge
Changed lines of the file:
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@@
 	(paper "A4")
 	(title_block
-		(title "Drako")
+		(title "Drako Hardware Challenge")
 		(date "2025-01-03")
 		(rev "1")
-		(company "Quarter Project")
-		(comment 1 "Access Controls & Covert Channels")
-		(comment 2 "CyberStorm Challenge")
+		(comment 1 "Drako Schematic")
+		(comment 2 "Cyberstorm 2025")
 	)
 	(junction
@@
 	)
 	(junction
+		(at 45.72 115.57)
+		(diameter 0)
+		(color 0 0 0 0)
+	)
+	(junction
 		(at 92.71 77.47)
 		(diameter 0)
@@
 	)
 	(junction
-		(at 45.72 46.99)
-		(diameter 0)
-		(color 0 0 0 0)
-	)
-	(junction
 		(at 44.45 49.53)
 		(diameter 0)
@@
 	)
 	(junction
-		(at 45.72 115.57)
-		(diameter 0)
-		(color 0 0 0 0)
-	)
-	(junction
 		(at 48.26 90.17)
 		(diameter 0)
@@
 	(wire
 		(pts
-			(xy 45.72 46.99) (xy 50.8 46.99)
+			(xy 27.94 46.99) (xy 50.8 46.99)
 		)
 		(stroke
@@
 	(wire
 		(pts
+			(xy 45.72 105.41) (xy 93.98 105.41)
+		)
+		(stroke
+			(width 0)
+			(type default)
+		)
+	)
+	(wire
+		(pts
 			(xy 144.78 149.86) (xy 144.78 118.11)
 		)
@@
 	(wire
 		(pts
-			(xy 45.72 46.99) (xy 45.72 115.57)
-		)
-		(stroke
-			(width 0)
-			(type default)
-		)
-	)
-	(wire
-		(pts
 			(xy 106.68 142.24) (xy 106.68 125.73)
 		)
@@
 	(wire
 		(pts
-			(xy 27.94 46.99) (xy 45.72 46.99)
+			(xy 45.72 115.57) (xy 45.72 105.41)
 		)
 		(stroke
 			(width 0)
 			(type default)
-			(color 236 209 14 1)
 		)
 	)
@@
 	(wire
 		(pts
+			(xy 86.36 67.31) (xy 93.98 67.31)
+		)
+		(stroke
+			(width 0)
+			(type default)
+		)
+	)
+	(wire
+		(pts
 			(xy 48.26 52.07) (xy 50.8 52.07)
 		)
@@
 	(wire
 		(pts
+			(xy 93.98 105.41) (xy 93.98 67.31)
+		)
+		(stroke
+			(width 0)
+			(type default)
+		)
+	)
+	(wire
+		(pts
 			(xy 48.26 101.6) (xy 48.26 90.17)
 		)
@@
 			)
 		)
-		(property "Value" "250Ω"
+		(property "Value" "47Ω"
 			(at 153.67 160.02 0)
 			(effects
@@
 		)
 		(instances
-			(project "TheGoldfish"
+			(project "drako-cyberstorm"
 				(path "/5a2f8960-3a2d-4fb3-8f1d-31afa13e1135"
 					(reference "R1")
@@
 		)
 		(instances
-			(project "TheGoldfish"
+			(project "drako-cyberstorm"
 				(path "/5a2f8960-3a2d-4fb3-8f1d-31afa13e1135"
 					(reference "U1")
@@
 		)
 		(instances
-			(project "TheGoldfish"
+			(project "drako-cyberstorm"
 				(path "/5a2f8960-3a2d-4fb3-8f1d-31afa13e1135"
 					(reference "U4")
@@
 		)
 		(instances
-			(project "TheGoldfish"
+			(project "drako-cyberstorm"
 				(path "/5a2f8960-3a2d-4fb3-8f1d-31afa13e1135"
 					(reference "U3")
@@
 		)
 		(instances
-			(project "TheGoldfish"
+			(project "drako-cyberstorm"
 				(path "/5a2f8960-3a2d-4fb3-8f1d-31afa13e1135"
 					(reference "U2")
@@
 		)
 		(instances
-			(project "TheGoldfish"
+			(project "drako-cyberstorm"
 				(path "/5a2f8960-3a2d-4fb3-8f1d-31afa13e1135"
 					(reference "Dual-7-Seg1")
